File: knob/knob.kicad_sch (KiCad schematic)
At the start: 12 parts, among them SW1 SW_Push, SW2 SW_Push, SW3 SW_Push, SW4 SW_Push, SW5 SW_Push, SW6 SW_Push, SW7 RotaryEncoder_Switch, SW8 RotaryEncoder_Switch, U1 TP4056-42-ESOP8

Commit message: sync
Parts:
- removed BT1: Battery_Cell, Connector_PinHeader_1.00mm:PinHeader_1x02_P1.00mm_Horizontal, symbol Device:Battery_Cell
- removed U1: TP4056-42-ESOP8, Package_SO:SOIC-8-1EP_3.9x4.9mm_P1.27mm_EP2.41x3.3mm_ThermalVias, symbol Battery_Management:TP4056-42-ESOP8
Changed lines of the file:
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@@
 	(wire
 		(pts
-			(xy 224.79 54.61) (xy 242.57 54.61)
+			(xy 168.91 85.09) (xy 168.91 83.82)
 		)
 		(stroke
@@
 	(wire
 		(pts
-			(xy 168.91 85.09) (xy 168.91 83.82)
+			(xy 191.77 83.82) (xy 191.77 85.09)
 		)
 		(stroke
@@
 	(wire
 		(pts
-			(xy 191.77 83.82) (xy 191.77 85.09)
+			(xy 100.33 93.98) (xy 100.33 100.33)
 		)
 		(stroke
@@
 		)
 	)
-	(wire
-		(pts
-			(xy 100.33 93.98) (xy 100.33 100.33)
-		)
-		(stroke
-			(width 0)
-			(type default)
-		)
-	)
 	(global_label "C"
 		(shape input)
@@
 	)
 	(symbol
-		(lib_id "Device:Battery_Cell")
-		(at 242.57 59.69 0)
-		(unit 1)
-		(exclude_from_sim no)
-		(in_bom yes)
-		(on_board yes)
-		(dnp no)
-		(fields_autoplaced yes)
-		(property "Reference" "BT1"
-			(at 246.38 56.5784 0)
-			(effects
-				(font
-					(size 1.27 1.27)
-				)
-				(justify left)
-			)
-		)
-		(property "Value" "Battery_Cell"
-			(at 246.38 59.1184 0)
-			(effects
-				(font
-					(size 1.27 1.27)
-				)
-				(justify left)
-			)
-		)
-		(property "Footprint" "Connector_PinHeader_1.00mm:PinHeader_1x02_P1.00mm_Horizontal"
-			(at 242.57 58.166 90)
-			(effects
-				(font
-					(size 1.27 1.27)
-				)
-				(hide yes)
-			)
-		)
-		(property "Datasheet" "~"
-			(at 242.57 58.166 90)
-			(effects
-				(font
-					(size 1.27 1.27)
-				)
-				(hide yes)
-			)
-		)
-		(property "Description" "Single-cell battery"
-			(at 242.57 59.69 0)
-			(effects
-				(font
-					(size 1.27 1.27)
-				)
-				(hide yes)
-			)
-		)
-		(pin "1"
-		)
-		(pin "2"
-		)
-		(instances
-			(project ""
-				(path "/d4f101b5-2d9a-42a4-8162-6f864c46b9d7"
-					(reference "BT1")
-					(unit 1)
-				)
-			)
-		)
-	)
-	(symbol
 		(lib_id "power:GND")
 		(at 91.44 91.44 90)
@@
 					(unit 1)
 				)
-			)
-		)
-	)
-	(symbol
-		(lib_id "Battery_Management:TP4056-42-ESOP8")
-		(at 214.63 59.69 0)
-		(unit 1)
-		(exclude_from_sim no)
-		(in_bom yes)
-		(on_board yes)
-		(dnp no)
-		(fields_autoplaced yes)
-		(property "Reference" "U1"
-			(at 216.7733 44.45 0)
-			(effects
-				(font
-					(size 1.27 1.27)
-				)
-				(justify left)
-			)
-		)
-		(property "Value" "TP4056-42-ESOP8"
-			(at 216.7733 46.99 0)
-			(effects
-				(font
-					(size 1.27 1.27)
-				)
-				(justify left)
-			)
-		)
-		(property "Footprint" "Package_SO:SOIC-8-1EP_3.9x4.9mm_P1.27mm_EP2.41x3.3mm_ThermalVias"
-			(at 215.138 82.55 0)
-			(effects
-				(font
-					(size 1.27 1.27)
-				)
-				(hide yes)
-			)
-		)
-		(property "Datasheet" "https://www.lcsc.com/datasheet/lcsc_datasheet_2410121619_TOPPOWER-Nanjing-Extension-Microelectronics-TP4056-42-ESOP8_C16581.pdf"
-			(at 214.63 85.09 0)
-			(effects
-				(font
-					(size 1.27 1.27)
-				)
-				(hide yes)
-			)
-		)
-		(property "Description" "1A Standalone Linear Li-ion/LiPo single-cell battery charger, 4.2V ±1% charge voltage, VCC = 4.0..8.0V, SOIC-8 (SOP-8)"
-			(at 215.138 80.01 0)
-			(effects
-				(font
-					(size 1.27 1.27)
-				)
-				(hide yes)
-			)
-		)
-		(pin "8"
-		)
-		(pin "9"
-		)
-		(pin "1"
-		)
-		(pin "5"
-		)
-		(pin "2"
-		)
-		(pin "4"
-		)
-		(pin "3"
-		)
-		(pin "6"
-		)
-		(pin "7"
-		)
-		(instances
-			(project ""
-				(path "/d4f101b5-2d9a-42a4-8162-6f864c46b9d7"
-					(reference "U1")
-					(unit 1)
-				)

Commit message: sync
Parts:
- removed A1: RaspberryPi_Pico, Module:RaspberryPi_Pico_Common_Unspecified, symbol MCU_Module:RaspberryPi_Pico
- removed SW1, SW2, SW3, SW4, SW5, SW6: SW_Push, Button_Switch_Keyboard:SW_Cherry_MX_1.00u_PCB, symbol Switch:SW_Push
- removed SW7, SW8: RotaryEncoder_Switch, Rotary_Encoder:RotaryEncoder_Alps_EC11E-Switch_Vertical_H20mm_MountingHoles, symbol Device:RotaryEncoder_Switch
- added D1, D2, D3, D4, D5, D6: SK6812MINI, cheyao macropad main PCB-third_party_neopixel.petty:SK6812MINI-E, symbol LED:SK6812MINI
- added U1: XIAO-RP2040-SMD, Seeed Studio XIAO Series Library:XIAO-RP2040-SMD, symbol Seeed_Studio_XIAO_Series:XIAO-RP2040-SMD
Connections:
- net A: now also U1.4 (GPIO29_A3_D3)
- net B: now also U1.1 (GPIO26_A0_D0)
- net C: now also U1.2 (GPIO27_A1_D1)
- net D: now also U1.6 (GPIO7_D5_SCL)
- net ENC0A: now also U1.5 (GPIO6_D4_SDA)
- net ENC0B: now also U1.8 (GPIO1_D7_CSn_RX)
- net GND: now also D1.2 (VSS), D2.2 (VSS), D3.2 (VSS), D4.2 (VSS), D5.2 (VSS), D6.2 (VSS), U1.13 (GND)
- net PUSH: now also U1.3 (GPIO28_A2_D2)
- new net: D4.1 (DOUT), D5.3 (DIN)
- new net: D3.1 (DOUT), D4.3 (DIN)
- new net: D2.1 (DOUT), D3.3 (DIN)
- new net: D1.1 (DOUT), D2.3 (DIN)
- new net: D5.1 (DOUT), D6.3 (DIN)
- new net +5V: D1.4 (VDD), D2.4 (VDD), D3.4 (VDD), D4.4 (VDD), D5.4 (VDD), D6.4 (VDD), U1.14 (5V)
- new net rgb: D1.3 (DIN), U1.7 (GPIO0_D6_TX)
- no-connect marks 9 -> 2
